Commit message: simple simulation

File: description/camera_only.urdf.xacro (robot description, xacro)
@@ -1,8 +1,18 @@
 <?xml version="1.0"?>
-<robot xmlns:xacro="http://www.ros.org/wiki/xacro" >
+<robot xmlns:xacro="http://www.ros.org/wiki/xacro" name="camera_only">
+    <!-- Base Link (world에 고정) -->
+    <link name="world"/>
+    <joint name="world_fixed" type="fixed">
+        <parent link="world"/>
+        <child link="base_link"/>
+        <origin xyz="0 0 0" rpy="0 0 0"/>
+    </joint>
+    <link name="base_link"/>
+    <!-- Camera Link -->
     <joint name="camera_joint" type="fixed">
-        <parent link="chassis"/>
+        <parent link="base_link"/>
         <child link="camera_link"/>
-        <origin xyz="0.276 0 0.181" rpy="0 0.18 0"/>
+        <!-- 카메라 위치 (높이 1m, 앞으로 0.5m) -->
+        <origin xyz="0.5 0 1.0" rpy="0 0.18 0"/>
     </joint>
     <link name="camera_link">
@@ -21,4 +31,5 @@
         </visual>
     </link>
+    <!-- Camera Optical Frame -->
     <joint name="camera_optical_joint" type="fixed">
         <parent link="camera_link"/>
@@ -26,11 +37,12 @@
         <origin xyz="0 0 0" rpy="${-pi/2} 0 ${-pi/2}"/>
     </joint>
-    <link name="camera_link_optical"></link>
+    <link name="camera_link_optical"/>
+    <!-- Gazebo Camera Sensor -->
     <gazebo reference="camera_link">
         <material>Gazebo/Black</material>
         <sensor name="camera" type="camera">
-            <pose> 0 0 0 0 0 0 </pose>
+            <pose>0 0 0 0 0 0</pose>
             <visualize>true</visualize>
-            <update_rate>10</update_rate>
+            <update_rate>30</update_rate>
             <camera>
                 <horizontal_fov>1.089</horizontal_fov>
@@ -46,5 +58,10 @@
             </camera>
             <plugin name="camera_controller" filename="libgazebo_ros_camera.so">
+                <ros>
+                    <namespace>/camera</namespace>
+                </ros>
                 <frame_name>camera_link_optical</frame_name>
+                <min_depth>0.1</min_depth>
+                <max_depth>100.0</max_depth>
             </plugin>
         </sensor>
